File: Hardware/LiPoBatteryBreadboardSupply.sch (EAGLE design)
At the start: 20 parts

Commit message: changes to the silkscreen and changes to the BOM
Parts:
- removed R4: 10k, resistor:R-US_R0402
- added R3: 100k, resistor:R-US_R0402
- added U$1: HANDLE.1HANDLE.025, CalvEngIO-Logos:HANDLE.1HANDLE.025
- C1, C2: device resistor:C-EUC0402 -> CalvEngIO-Passives:CAPACITOR0603
- C3: value 100pF -> 2.2u; device resistor:C-EUC0402 -> resistor:C-EUC0603
- C4: value 1u -> 2.2u
- C5: value 2.2u -> 100pF; device resistor:C-EUC0603 -> resistor:C-EUC0402
- U$6: value LOGO.08 -> HANDLE.1HANDLE.08; device CalvEngIO-Logo:LOGO.08 -> CalvEngIO-Logos:HANDLE.1HANDLE.08
- renumbered PWR to VDD
Connections:
- removed net N$3: 3V3.SWITCH.3, 3V3.SWITCH.5, 3V3.SWITCH.6, 3V3.SWITCH.7, R4.2
- net 3.3V: now also C3.1; no longer C5.1
- net EN: now also R3.2
- net GND: now also R3.1; no longer R4.1
- net N$4: now also C5.1; no longer C3.1
Other:
- note added: "Rev 0.3"
- moved on the sheet: C3, C5
Changed lines of the file:
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@@
 <?xml version="1.0" encoding="utf-8"?>
 <!DOCTYPE eagle SYSTEM "eagle.dtd">
-<eagle version="7.3.0">
+<eagle version="8.1.1">
 <drawing>
 <settings>
@@
 <part name="SUPPLY3" library="SparkFun-PowerSymbols" deviceset="V_BATT" device=""/>
 <part name="GND3" library="SparkFun-PowerSymbols" deviceset="GND" device=""/>
-<part name="C1" library="resistor" deviceset="C-EU" device="C0402" value="100n"/>
-<part name="C2" library="resistor" deviceset="C-EU" device="C0402" value="100n"/>
+<part name="C1" library="CalvEngIO-Passives" deviceset="CAPACITOR" device="0603" value="100n"/>
+<part name="C2" library="CalvEngIO-Passives" deviceset="CAPACITOR" device="0603" value="100n"/>
 <part name="GND4" library="SparkFun-PowerSymbols" deviceset="GND" device=""/>
 <part name="GND5" library="SparkFun-PowerSymbols" deviceset="GND" device=""/>
@@
 <part name="SUPPLY4" library="SparkFun-PowerSymbols" deviceset="V_BATT" device=""/>
 <part name="GND6" library="SparkFun-PowerSymbols" deviceset="GND" device=""/>
-<part name="C3" library="resistor" deviceset="C-EU" device="C0402" value="100pF"/>
+<part name="C5" library="resistor" deviceset="C-EU" device="C0402" value="100pF"/>
 <part name="GND7" library="SparkFun-PowerSymbols" deviceset="GND" device=""/>
-<part name="C4" library="resistor" deviceset="C-EU" device="C0603" value="1u"/>
+<part name="C4" library="resistor" deviceset="C-EU" device="C0603" value="2.2u"/>
 <part name="J1" library="SparkFun-Connectors" deviceset="CONN_03" device=""/>
 <part name="SUPPLY6" library="SparkFun-PowerSymbols" deviceset="V_BATT" device=""/>
@@
 <part name="SUPPLY1" library="SparkFun-PowerSymbols" deviceset="VDD" device=""/>
 <part name="SUPPLY2" library="SparkFun-PowerSymbols" deviceset="VDD" device=""/>
-<part name="C5" library="resistor" deviceset="C-EU" device="C0603" value="2.2u"/>
+<part name="C3" library="resistor" deviceset="C-EU" device="C0603" value="2.2u"/>
 <part name="GND8" library="SparkFun-PowerSymbols" deviceset="GND" device=""/>
 <part name="SUPPLY5" library="SparkFun-PowerSymbols" deviceset="3.3V" device=""/>
-<part name="PWR" library="CalvEngIO-LED" deviceset="LED" device="0603"/>
+<part name="VDD" library="CalvEngIO-LED" deviceset="LED" device="0603"/>
 <part name="3.3V" library="CalvEngIO-LED" deviceset="LED" device="0603"/>
 <part name="GND9" library="SparkFun-PowerSymbols" deviceset="GND" device=""/>
@@
 <part name="3V3.SWITCH" library="CalvEngIO-Switches" deviceset="SWITCH.JS202011JCQN" device=""/>
 <part name="SUPPLY12" library="SparkFun-PowerSymbols" deviceset="V_BATT" device=""/>
-<part name="U$6" library="CalvEngIO-Logo" deviceset="LOGO.08" device=""/>
-<part name="R4" library="resistor" deviceset="R-US_" device="R0402" value="10k"/>
+<part name="U$6" library="CalvEngIO-Logos" deviceset="HANDLE.1" device="HANDLE.08"/>
+<part name="R3" library="resistor" deviceset="R-US_" device="R0402" value="100k"/>
 <part name="GND12" library="SparkFun-PowerSymbols" deviceset="GND" device=""/>
 <part name="J2" library="CalvEngIO-Connectors" deviceset="JMP.03X2" device="HEADERS"/>
@@
 <part name="FD1" library="adafruit" deviceset="FIDUCIAL" device=""/>
 <part name="FD2" library="adafruit" deviceset="FIDUCIAL" device=""/>
+<part name="U$1" library="CalvEngIO-Logos" deviceset="HANDLE.1" device="HANDLE.025" value="HANDLE.1HANDLE.025"/>
 </parts>
 <sheets>
@@
 <wire x1="142.24" y1="-2.54" x2="-53.34" y2="-2.54" width="0.635" layer="94"/>
 <wire x1="-53.34" y1="-2.54" x2="-53.34" y2="101.6" width="0.635" layer="94"/>
+<text x="60.96" y="104.14" size="2.54" layer="91">Rev 0.3</text>
 </plain>
 <instances>
@@
 <instance part="SUPPLY3" gate="G$1" x="-27.94" y="78.74"/>
 <instance part="GND3" gate="1" x="-38.1" y="66.04"/>
-<instance part="C1" gate="G$1" x="-2.54" y="73.66" rot="R180"/>
-<instance part="C2" gate="G$1" x="30.48" y="73.66" rot="R180"/>
+<instance part="C1" gate="G$1" x="-2.54" y="76.2" rot="R180"/>
+<instance part="C2" gate="G$1" x="30.48" y="76.2" rot="R180"/>
 <instance part="GND4" gate="1" x="-2.54" y="66.04"/>
 <instance part="GND5" gate="1" x="30.48" y="66.04"/>
@@
 <instance part="SUPPLY4" gate="G$1" x="-27.94" y="48.26"/>
 <instance part="GND6" gate="1" x="-38.1" y="25.4"/>
-<instance part="C3" gate="G$1" x="7.62" y="30.48"/>
+<instance part="C5" gate="G$1" x="7.62" y="30.48"/>
 <instance part="GND7" gate="1" x="7.62" y="20.32"/>
 <instance part="C4" gate="G$1" x="-43.18" y="35.56" rot="R180"/>
@@
 <instance part="SUPPLY1" gate="VDD" x="0" y="83.82"/>
 <instance part="SUPPLY2" gate="VDD" x="33.02" y="83.82"/>
-<instance part="C5" gate="G$1" x="17.78" y="40.64"/>
+<instance part="C3" gate="G$1" x="17.78" y="40.64"/>
 <instance part="GND8" gate="1" x="17.78" y="30.48"/>
 <instance part="SUPPLY5" gate="G$1" x="7.62" y="48.26"/>
-<instance part="PWR" gate="G$1" x="104.14" y="73.66"/>
+<instance part="VDD" gate="G$1" x="104.14" y="73.66"/>
 <instance part="3.3V" gate="G$1" x="-27.94" y="15.24"/>
 <instance part="GND9" gate="1" x="-27.94" y="5.08"/>
@@
 <instance part="SUPPLY12" gate="G$1" x="38.1" y="43.18"/>
 <instance part="U$6" gate="G$1" x="76.2" y="25.4"/>
-<instance part="R4" gate="G$1" x="55.88" y="17.78" rot="R90"/>
-<instance part="GND12" gate="1" x="55.88" y="7.62"/>
+<instance part="R3" gate="G$1" x="58.42" y="35.56" rot="R90"/>
+<instance part="GND12" gate="1" x="58.42" y="25.4"/>
 <instance part="J2" gate="G$1" x="10.16" y="78.74"/>
 <instance part="J3" gate="G$1" x="43.18" y="78.74"/>
@@
 <instance part="FD1" gate="G$1" x="76.2" y="48.26"/>
 <instance part="FD2" gate="G$1" x="83.82" y="43.18"/>
+<instance part="U$1" gate="G$1" x="76.2" y="30.48"/>
 </instances>
 <busses>
@@
 <pinref part="C1" gate="G$1" pin="1"/>
 <pinref part="GND4" gate="1" pin="GND"/>
-<wire x1="-2.54" y1="68.58" x2="-2.54" y2="71.12" width="0.1524" layer="91"/>
+<wire x1="-2.54" y1="71.12" x2="-2.54" y2="68.58" width="0.1524" layer="91"/>
 </segment>
 <segment>
 <pinref part="C2" gate="G$1" pin="1"/>
 <pinref part="GND5" gate="1" pin="GND"/>
-<wire x1="30.48" y1="68.58" x2="30.48" y2="71.12" width="0.1524" layer="91"/>
+<wire x1="30.48" y1="71.12" x2="30.48" y2="68.58" width="0.1524" layer="91"/>
 </segment>
 <segment>
@@
 </segment>
 <segment>
-<pinref part="C3" gate="G$1" pin="2"/>
+<pinref part="C5" gate="G$1" pin="2"/>
 <pinref part="GND7" gate="1" pin="GND"/>
 <wire x1="7.62" y1="22.86" x2="7.62" y2="25.4" width="0.1524" layer="91"/>
 </segment>
 <segment>
-<pinref part="C5" gate="G$1" pin="2"/>
+<pinref part="C3" gate="G$1" pin="2"/>
 <pinref part="GND8" gate="1" pin="GND"/>
 <wire x1="17.78" y1="33.02" x2="17.78" y2="35.56" width="0.1524" layer="91"/>
@@
 </segment>
 <segment>
-<pinref part="PWR" gate="G$1" pin="C"/>
+<pinref part="VDD" gate="G$1" pin="C"/>
 <pinref part="GND10" gate="1" pin="GND"/>
 <wire x1="104.14" y1="66.04" x2="104.14" y2="68.58" width="0.1524" layer="91"/>
 </segment>
 <segment>
-<pinref part="R4" gate="G$1" pin="1"/>
+<pinref part="R3" gate="G$1" pin="1"/>
 <pinref part="GND12" gate="1" pin="GND"/>
-<wire x1="55.88" y1="10.16" x2="55.88" y2="12.7" width="0.1524" layer="91"/>
+<wire x1="58.42" y1="27.94" x2="58.42" y2="30.48" width="0.1524" layer="91"/>
 </segment>
 </net>
@@
 <segment>
 <pinref part="LDO" gate="G$1" pin="BYP/ADJ"/>
-<pinref part="C3" gate="G$1" pin="1"/>
+<pinref part="C5" gate="G$1" pin="1"/>
 <wire x1="5.08" y1="35.56" x2="7.62" y2="35.56" width="0.1524" layer="91"/>
 <wire x1="7.62" y1="35.56" x2="7.62" y2="33.02" width="0.1524" layer="91"/>
@@
 <wire x1="5.08" y1="40.64" x2="7.62" y2="40.64" width="0.1524" layer="91"/>
 <wire x1="7.62" y1="40.64" x2="7.62" y2="45.72" width="0.1524" layer="91"/>
-<pinref part="C5" gate="G$1" pin="1"/>
+<pinref part="C3" gate="G$1" pin="1"/>
 <wire x1="7.62" y1="45.72" x2="7.62" y2="48.26" width="0.1524" layer="91"/>
 <wire x1="17.78" y1="43.18" x2="17.78" y2="45.72" width="0.1524" layer="91"/>
@@
 <net name="N$2" class="0">
 <segment>
-<pinref part="PWR" gate="G$1" pin="A"/>
+<pinref part="VDD" gate="G$1" pin="A"/>
 <pinref part="R1" gate="G$1" pin="1"/>
 <wire x1="104.14" y1="78.74" x2="104.14" y2="76.2" width="0.1524" layer="91"/>
@@
 <segment>
 <pinref part="3V3.SWITCH" gate="G$1" pin="1"/>
-<wire x1="53.34" y1="43.18" x2="55.88" y2="43.18" width="0.1524" layer="91"/>
-<label x="55.88" y="43.18" size="1.27" layer="95" xref="yes"/>
-</segment>
-</net>
-<net name="N$3" class="0">
-<segment>
-<pinref part="3V3.SWITCH" gate="G$1" pin="6"/>
-<wire x1="43.18" y1="33.02" x2="40.64" y2="33.02" width="0.1524" layer="91"/>
-<wire x1="40.64" y1="33.02" x2="40.64" y2="25.4" width="0.1524" layer="91"/>
-<pinref part="3V3.SWITCH" gate="G$1" pin="7"/>
-<pinref part="R4" gate="G$1" pin="2"/>
-<wire x1="53.34" y1="30.48" x2="55.88" y2="30.48" width="0.1524" layer="91"/>
-<wire x1="55.88" y1="30.48" x2="55.88" y2="25.4" width="0.1524" layer="91"/>
-<pinref part="3V3.SWITCH" gate="G$1" pin="5"/>
-<wire x1="55.88" y1="25.4" x2="55.88" y2="22.86" width="0.1524" layer="91"/>
-<wire x1="53.34" y1="35.56" x2="55.88" y2="35.56" width="0.1524" layer="91"/>
-<wire x1="55.88" y1="35.56" x2="55.88" y2="30.48" width="0.1524" layer="91"/>
-<junction x="55.88" y="30.48"/>
-<pinref part="3V3.SWITCH" gate="G$1" pin="3"/>
-<wire x1="53.34" y1="38.1" x2="55.88" y2="38.1" width="0.1524" layer="91"/>
-<wire x1="55.88" y1="38.1" x2="55.88" y2="35.56" width="0.1524" layer="91"/>
-<junction x="55.88" y="35.56"/>
-<wire x1="40.64" y1="25.4" x2="55.88" y2="25.4" width="0.1524" layer="91"/>
-<junction x="55.88" y="25.4"/>
-</segment>
-</net>
+<wire x1="53.34" y1="43.18" x2="58.42" y2="43.18" width="0.1524" layer="91"/>
+<label x="60.96" y="43.18" size="1.27" layer="95" xref="yes"/>
+<pinref part="R3" gate="G$1" pin="2"/>
+<wire x1="58.42" y1="43.18" x2="60.96" y2="43.18" width="0.1524" layer="91"/>
+<wire x1="58.42" y1="40.64" x2="58.42" y2="43.18" width="0.1524" layer="91"/>
+<junction x="58.42" y="43.18"/>
+</segment>
+</net>

Commit message: changes to BOM and change in value of Cbypass on regulator in schematic
Parts:
- C5: value 100pF -> 47pF
Changed lines of the file:
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@@
 <part name="SUPPLY4" library="SparkFun-PowerSymbols" deviceset="V_BATT" device=""/>
 <part name="GND6" library="SparkFun-PowerSymbols" deviceset="GND" device=""/>
-<part name="C5" library="resistor" deviceset="C-EU" device="C0402" value="100pF"/>
+<part name="C5" library="resistor" deviceset="C-EU" device="C0402" value="47pF"/>
 <part name="GND7" library="SparkFun-PowerSymbols" deviceset="GND" device=""/>
 <part name="C4" library="resistor" deviceset="C-EU" device="C0603" value="2.2u"/>
